File: kgiu/kicad.kicad_pcb (KiCad board)
At the start: 2 copper layers, 65 x 56 mm, 24 parts, among them J1 OSTTC020162, J2 Raspberry_Pi_2_3, J3 OSTTC020162, Q1 STP55NF06L, SW1 206-2ST, U1 CD4050BE, U2 4N35, U3 4N35, U4 4N35

Commit message: fixed pcb footprint for OSTTC020162
Parts:
- moved J3 0.84 mm to (101.0, 122.6)
- moved J1 0.63 mm to (114.3, 122.6)
Changed lines of the file:
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@@
-(kicad_pcb (version 20171130) (host pcbnew 5.1.2-f72e74a~84~ubuntu18.04.1)
+(kicad_pcb (version 20171130) (host pcbnew 5.1.3-ffb9f22~84~ubuntu18.04.1)
   (general
     (thickness 1.6)
@@
   (title_block
     (title "Keybus to GPIO Interface Unit")
-    (date 2019-07-14)
-    (rev 1)
+    (date 2019-07-30)
+    (rev 1.1)
     (comment 1 "Designed by Lindo St. Angel")
     (comment 2 "Part of the ALL Project - See https://github.com/goruck/all for more information.")
@@
     (add_net GNDD)
   )
+  (module digikey-footprints:Term_Block_1x2_P5mm (layer F.Cu)
+    (at 100.965 122.555)
+    (descr http://www.on-shore.com/wp-content/uploads/2015/09/osttcxx0162.pdf)
+    (fp_text reference J3 (at 2.7 -4.8) (layer F.SilkS)
+      (effects (font (size 1 1) (thickness 0.15)))
+    )
+    (fp_text value OSTTC020162 (at 2.05 5.05) (layer F.Fab)
+      (effects (font (size 1 1) (thickness 0.15)))
+    )
+    (fp_line (start -2.5 -3.75) (end -2.5 3.75) (layer F.Fab) (width 0.1))
+    (fp_line (start -2.75 -4) (end -2.75 4) (layer F.CrtYd) (width 0.05))
+    (fp_line (start 7.5 -3.75) (end -2.5 -3.75) (layer F.Fab) (width 0.1))
+    (fp_line (start 7.5 3.75) (end -2.5 3.75) (layer F.Fab) (width 0.1))
+    (fp_line (start 7.5 -3.75) (end 7.5 3.75) (layer F.Fab) (width 0.1))
+    (fp_line (start -2.75 4) (end 7.75 4) (layer F.CrtYd) (width 0.05))
+    (fp_line (start 7.75 -4) (end 7.75 4) (layer F.CrtYd) (width 0.05))
+    (fp_line (start -2.75 -4) (end 7.75 -4) (layer F.CrtYd) (width 0.05))
+    (fp_line (start 7.6 -3.85) (end 7.1 -3.85) (layer F.SilkS) (width 0.1))
+    (fp_line (start 7.6 -3.85) (end 7.6 -3.4) (layer F.SilkS) (width 0.1))
+    (fp_line (start -2.6 -3.85) (end -2.6 -3.4) (layer F.SilkS) (width 0.1))
+    (fp_line (start -2.6 -3.85) (end -2.1 -3.85) (layer F.SilkS) (width 0.1))
+    (fp_line (start -2.6 3.85) (end -2.1 3.85) (layer F.SilkS) (width 0.1))
+    (fp_line (start -2.6 3.85) (end -2.6 3.35) (layer F.SilkS) (width 0.1))
+    (fp_line (start 7.6 3.85) (end 7.6 3.35) (layer F.SilkS) (width 0.1))
+    (fp_line (start 7.6 3.85) (end 7.1 3.85) (layer F.SilkS) (width 0.1))
+    (fp_text user %R (at 2.5 0) (layer F.Fab)
+      (effects (font (size 1 1) (thickness 0.15)))
+    )
+    (pad 2 thru_hole circle (at 5 0) (size 2.5 2.5) (drill 1.3) (layers *.Cu *.Mask)
+      (net 32 "Net-(J3-Pad2)"))
+    (pad 1 thru_hole rect (at 0 0) (size 2.5 2.5) (drill 1.3) (layers *.Cu *.Mask)
+      (net 33 "Net-(J3-Pad1)"))
+  )
+  (module digikey-footprints:Term_Block_1x2_P5mm (layer F.Cu)
+    (at 114.3 122.555)
+    (descr http://www.on-shore.com/wp-content/uploads/2015/09/osttcxx0162.pdf)
+    (fp_text reference J1 (at 2.7 -4.8) (layer F.SilkS)
+      (effects (font (size 1 1) (thickness 0.15)))
+    )
+    (fp_text value OSTTC020162 (at 2.05 5.05) (layer F.Fab)
+      (effects (font (size 1 1) (thickness 0.15)))
+    )
+    (fp_line (start -2.5 -3.75) (end -2.5 3.75) (layer F.Fab) (width 0.1))
+    (fp_line (start -2.75 -4) (end -2.75 4) (layer F.CrtYd) (width 0.05))
+    (fp_line (start 7.5 -3.75) (end -2.5 -3.75) (layer F.Fab) (width 0.1))
+    (fp_line (start 7.5 3.75) (end -2.5 3.75) (layer F.Fab) (width 0.1))
+    (fp_line (start 7.5 -3.75) (end 7.5 3.75) (layer F.Fab) (width 0.1))
+    (fp_line (start -2.75 4) (end 7.75 4) (layer F.CrtYd) (width 0.05))
+    (fp_line (start 7.75 -4) (end 7.75 4) (layer F.CrtYd) (width 0.05))
+    (fp_line (start -2.75 -4) (end 7.75 -4) (layer F.CrtYd) (width 0.05))
+    (fp_line (start 7.6 -3.85) (end 7.1 -3.85) (layer F.SilkS) (width 0.1))
+    (fp_line (start 7.6 -3.85) (end 7.6 -3.4) (layer F.SilkS) (width 0.1))
+    (fp_line (start -2.6 -3.85) (end -2.6 -3.4) (layer F.SilkS) (width 0.1))
+    (fp_line (start -2.6 -3.85) (end -2.1 -3.85) (layer F.SilkS) (width 0.1))
+    (fp_line (start -2.6 3.85) (end -2.1 3.85) (layer F.SilkS) (width 0.1))
+    (fp_line (start -2.6 3.85) (end -2.6 3.35) (layer F.SilkS) (width 0.1))
+    (fp_line (start 7.6 3.85) (end 7.6 3.35) (layer F.SilkS) (width 0.1))
+    (fp_line (start 7.6 3.85) (end 7.1 3.85) (layer F.SilkS) (width 0.1))
+    (fp_text user %R (at 2.5 0) (layer F.Fab)
+      (effects (font (size 1 1) (thickness 0.15)))
+    )
+    (pad 2 thru_hole circle (at 5 0) (size 2.5 2.5) (drill 1.3) (layers *.Cu *.Mask)
+      (net 54 GNDA))
+    (pad 1 thru_hole rect (at 0 0) (size 2.5 2.5) (drill 1.3) (layers *.Cu *.Mask)
+      (net 29 +12V))
+  )
   (module Capacitor_THT:CP_Axial_L11.0mm_D6.0mm_P18.00mm_Horizontal (layer F.Cu)
     (at 126.49 123.825)
@@
     )
   )
-  (module digikey-footprints:Term_Block_1x2_P5mm (layer F.Cu)
-    (at 114.3 123.19)
-    (descr http://www.on-shore.com/wp-content/uploads/2015/09/osttcxx0162.pdf)
-    (fp_text reference J1 (at 2.7 -4.8) (layer F.SilkS)
-      (effects (font (size 1 1) (thickness 0.15)))
-    )
-    (fp_text value OSTTC020162 (at 2.05 5.05) (layer F.Fab)
-      (effects (font (size 1 1) (thickness 0.15)))
-    )
-    (fp_line (start -2.5 -3.75) (end -2.5 3.75) (layer F.Fab) (width 0.1))
-    (fp_line (start -2.75 -4) (end -2.75 4) (layer F.CrtYd) (width 0.05))
-    (fp_line (start 7.5 -3.75) (end -2.5 -3.75) (layer F.Fab) (width 0.1))
-    (fp_line (start 7.5 3.75) (end -2.5 3.75) (layer F.Fab) (width 0.1))
-    (fp_line (start 7.5 -3.75) (end 7.5 3.75) (layer F.Fab) (width 0.1))
-    (fp_line (start -2.75 4) (end 7.75 4) (layer F.CrtYd) (width 0.05))
-    (fp_line (start 7.75 -4) (end 7.75 4) (layer F.CrtYd) (width 0.05))
-    (fp_line (start -2.75 -4) (end 7.75 -4) (layer F.CrtYd) (width 0.05))
-    (fp_line (start 7.6 -3.85) (end 7.1 -3.85) (layer F.SilkS) (width 0.1))
-    (fp_line (start 7.6 -3.85) (end 7.6 -3.4) (layer F.SilkS) (width 0.1))
-    (fp_line (start -2.6 -3.85) (end -2.6 -3.4) (layer F.SilkS) (width 0.1))
-    (fp_line (start -2.6 -3.85) (end -2.1 -3.85) (layer F.SilkS) (width 0.1))
-    (fp_line (start -2.6 3.85) (end -2.1 3.85) (layer F.SilkS) (width 0.1))
-    (fp_line (start -2.6 3.85) (end -2.6 3.35) (layer F.SilkS) (width 0.1))
-    (fp_line (start 7.6 3.85) (end 7.6 3.35) (layer F.SilkS) (width 0.1))
-    (fp_line (start 7.6 3.85) (end 7.1 3.85) (layer F.SilkS) (width 0.1))
-    (fp_text user %R (at 2.5 0) (layer F.Fab)
-      (effects (font (size 1 1) (thickness 0.15)))
-    )
-    (pad 2 thru_hole circle (at 5 0) (size 1.524 1.524) (drill 0.762) (layers *.Cu *.Mask)
-      (net 54 GNDA))
-    (pad 1 thru_hole circle (at 0 0) (size 1.524 1.524) (drill 0.762) (layers *.Cu *.Mask)
-      (net 29 +12V))
-  )
-  (module digikey-footprints:Term_Block_1x2_P5mm (layer F.Cu)
-    (at 100.33 123.11)
-    (descr http://www.on-shore.com/wp-content/uploads/2015/09/osttcxx0162.pdf)
-    (fp_text reference J3 (at 2.7 -4.8) (layer F.SilkS)
-      (effects (font (size 1 1) (thickness 0.15)))
-    )
-    (fp_text value OSTTC020162 (at 2.05 5.05) (layer F.Fab)
-      (effects (font (size 1 1) (thickness 0.15)))
-    )
-    (fp_line (start -2.5 -3.75) (end -2.5 3.75) (layer F.Fab) (width 0.1))
-    (fp_line (start -2.75 -4) (end -2.75 4) (layer F.CrtYd) (width 0.05))
-    (fp_line (start 7.5 -3.75) (end -2.5 -3.75) (layer F.Fab) (width 0.1))
-    (fp_line (start 7.5 3.75) (end -2.5 3.75) (layer F.Fab) (width 0.1))
-    (fp_line (start 7.5 -3.75) (end 7.5 3.75) (layer F.Fab) (width 0.1))
-    (fp_line (start -2.75 4) (end 7.75 4) (layer F.CrtYd) (width 0.05))
-    (fp_line (start 7.75 -4) (end 7.75 4) (layer F.CrtYd) (width 0.05))
-    (fp_line (start -2.75 -4) (end 7.75 -4) (layer F.CrtYd) (width 0.05))
-    (fp_line (start 7.6 -3.85) (end 7.1 -3.85) (layer F.SilkS) (width 0.1))
-    (fp_line (start 7.6 -3.85) (end 7.6 -3.4) (layer F.SilkS) (width 0.1))
-    (fp_line (start -2.6 -3.85) (end -2.6 -3.4) (layer F.SilkS) (width 0.1))
-    (fp_line (start -2.6 -3.85) (end -2.1 -3.85) (layer F.SilkS) (width 0.1))
-    (fp_line (start -2.6 3.85) (end -2.1 3.85) (layer F.SilkS) (width 0.1))
-    (fp_line (start -2.6 3.85) (end -2.6 3.35) (layer F.SilkS) (width 0.1))
-    (fp_line (start 7.6 3.85) (end 7.6 3.35) (layer F.SilkS) (width 0.1))
-    (fp_line (start 7.6 3.85) (end 7.1 3.85) (layer F.SilkS) (width 0.1))
-    (fp_text user %R (at 2.5 0) (layer F.Fab)
-      (effects (font (size 1 1) (thickness 0.15)))
-    )
-    (pad 2 thru_hole circle (at 5 0) (size 1.524 1.524) (drill 0.762) (layers *.Cu *.Mask)
-      (net 32 "Net-(J3-Pad2)"))
-    (pad 1 thru_hole circle (at 0 0) (size 1.524 1.524) (drill 0.762) (layers *.Cu *.Mask)
-      (net 33 "Net-(J3-Pad1)"))
-  )
   (module Button_Switch_THT:SW_DIP_SPSTx02_Slide_9.78x7.26mm_W7.62mm_P2.54mm (layer F.Cu)
